File: KiCad/Motor_Power_Modul/Motor_Power_Modul.kicad_pcb (KiCad board)
At the start: 2 copper layers, 55 x 40 mm, 23 parts, among them J1 Power Input, J2 Power Out, J3 Power Out, J4 Motor Output, J5 Input, J6 Dead Man, Q1 IRF3708, Q2 IRF3708, U1 IR2302

Commit message: Iteration 2 von DC/DC Wandler
Parts:
- moved C1 16.7 mm to (103.7, 113.3)
- moved C2 2.54 mm to (104.1, 121.9)
- moved J3 0.25 mm to (120.4, 113.8)
Connections:
- R2 pad 2: Net-(U1-LO) -> unconnected-(R2-Pad2)
- U1 pad 5: Net-(U1-LO) -> unconnected-(U1-LO-Pad5)
Routing:
- net GND: track 184.5 -> 175.7 mm
- net Net-(U1-LO): track 5.56 -> 0.00 mm
- net (no net): track 0.00 -> 5.56 mm
- net VCC: track 225.2 -> 224.5 mm
Other:
- board text added: "453788"
- board text added: "V2"
